File: Circuit/SmartDoorKeeper.kicad_pcb (KiCad board)
At the start: 2 copper layers, 80 x 50 mm, 147 parts, among them J1 ServoOut, J2 LockDetect, J3 DoorSwitch, J4 +5V DC Input, J5 USB_OTG, J6 PN532_SPI, Q2 IRLML6344TRPbF, Q3 IRLML6344TRPbF, Q4 IRLML6344TRPbF, Q5 IRLML6344TRPbF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

Commit message: Smart Door Keyper -> Smart Door Keeperに変更
Other:
- board text added: "Smart Door Keeper"
- board text removed: "Smart Door Keyper"
Changed lines of the file:
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@@
     (effects (font (size 0.85 0.85) (thickness 0.15)))
   )
-  (gr_text "Smart Door Keyper" (at 75.5 84.75) (layer B.SilkS)
+  (gr_text "Smart Door Keeper" (at 75.5 84.75) (layer B.SilkS)
     (effects (font (size 1.5 1.5) (thickness 0.3)) (justify left mirror))
   )
